File: PCB/OpenFlipdisc.kicad_pcb (KiCad board)
At the start: 2 copper layers, 111.6 x 68.8 mm, 49 parts, among them J1 Barrel_Jack, J2 Screw_Terminal_01x05, J3 Screw_Terminal_01x05, J4 Conn_01x08, U1 R-78E5.0-1.0, U2 74HC595, U3 74HC595, U4 74HC595, U5 TB6612FNG, U6 TB6612FNG, U7 TB6612FNG, U8 TB6612FNG, U9 TB6612FNG

Commit message: MORE STUFF
Parts:
- A1: renamed from Pi Pico 2 W
- moved C13 0.50 mm to (124.8, 88.0)
- renumbered fuse to F1, CLEAR to SW1, FUNC1 to SW2, FUNC2 to SW3, RESET to SW4
Connections:
- D1 pad 1: Net-(D1-K) -> VM
- D1 pad 2: VM -> Net-(D1-A)
- F1 pad 2: Net-(D1-K) -> Net-(D1-A)
Routing:
- net Net-(D1-K): track 8.62 -> 0.00 mm
- net Net-(D1-A): track 0.00 -> 8.20 mm
- net +3V3: track 246.0 -> 254.0 mm
- net VM: track 184.6 -> 186.7 mm
- net GP10: track 99.0 -> 101.0 mm
- net DRV3_AIN1: track 21.4 -> 22.1 mm
- net DRV3_AIN2: track 10.8 -> 11.4 mm
- net GND: track 208.2 -> 208.7 mm
Other:
- board text added: "ACTIVE"
- board text added: "CLEAR"
- board text added: "FUNC1"
- board text added: "FUNC2"
- board text added: "NORMAL"
- board text added: "Open-FlipDisc"
- board text added: "fuse"
- board text added: "reset"
- board text added: "this is a PCB part of an open-source flip disc display module project ie- Open-FlipDisc.. made by: https://shashwat.cc"
- board text added: "⇑ a smiling flipdot grid"

Commit message: added all production files
Parts:
- C1: footprint Capacitor_THT:CP_Radial_D8.0mm_P3.50mm -> Capacitor_THT:CP_Radial_D10.0mm_P5.00mm
- moved C1 0.25 mm to (137.0, 106.8)
Other:
- board text added: "RESET"
- board text removed: "reset"

Commit message: replaced RECOM with AP63205WU-7 for better availability
Parts:
- added C19: 22uF, Capacitor_SMD:C_1206_3216Metric, F.Cu at (159.8, 97.0)
- added C20: 100nF, Capacitor_SMD:C_0805_2012Metric, F.Cu at (160.5, 92.0)
- added L1: 4.7uH, Inductor_SMD:L_Sunlord_SWPA5040S, F.Cu at (164.5, 97.2)
- U1: value R-78E5.0-1.0 -> AP63205WU-7; footprint Converter_DCDC:Converter_DCDC_RECOM_R-78E-0.5_THT -> OpenFlipdisc_EasyEDA:TSOT-23-6_L2.9-W1.6-P0.95-LS2.8-BL
- moved C5 8.80 mm to (156.8, 97.0), turned to -90 degrees
- moved U1 1.72 mm to (164.5, 92.0), turned to 90 degrees
Connections:
- U1 pad 1: VM -> +5V
- U1 pad 2: GND -> VM
- U1 pad 3: +5V -> VM
Routing:
- net +5V: track 67.8 -> 94.2 mm
- net VM: track 186.7 -> 200.3 mm, vias 1 -> 2
- net Net-(U1-SW): track 0.00 -> 10.2 mm
- net Net-(U1-BST): track 0.00 -> 2.80 mm
- net GP10: track 101.0 -> 102.2 mm
