File: PCB/OpenFlipdisc.kicad_sch (KiCad schematic)
At the start: 48 parts, among them J1 Barrel_Jack, J2 Screw_Terminal_01x05, J3 Screw_Terminal_01x05, J4 Conn_01x08, SW1 CLEAR, SW2 FUNC1, SW3 FUNC2, SW4 RESET, U1 R-78E5.0-1.0, U2 74HC595, U3 74HC595, U4 74HC595, U5 TB6612FNG, U6 TB6612FNG, U7 TB6612FNG, U8 TB6612FNG, U9 TB6612FNG

Commit message: MORE STUFF
Connections:
- net VM: now also D1.1 (K); no longer D1.2 (A)
- net at F1.2: now also D1.2 (A); no longer D1.1 (K)
Other:
- moved on the sheet: D1
Changed lines of the file:
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@@
 	(symbol
 		(lib_id "Device:D_Schottky")
-		(at 48.26 180.34 0)
+		(at 48.26 180.34 180)
 		(unit 1)
 		(body_style 1)
@@
 		(fields_autoplaced yes)
 		(property "Reference" "D1"
-			(at 47.9425 173.99 0)
+			(at 48.5775 173.99 0)
 			(show_name no)
 			(do_not_autoplace no)
@@
 		)
 		(property "Value" "SS34"
-			(at 47.9425 176.53 0)
+			(at 48.5775 176.53 0)
 			(show_name no)
 			(do_not_autoplace no)

Commit message: added all production files
Parts:
- C1: footprint Capacitor_THT:CP_Radial_D8.0mm_P3.50mm -> Capacitor_THT:CP_Radial_D10.0mm_P5.00mm
Changed lines of the file:
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@@
 			)
 		)
-		(property "Footprint" "Capacitor_THT:CP_Radial_D8.0mm_P3.50mm"
+		(property "Footprint" "Capacitor_THT:CP_Radial_D10.0mm_P5.00mm"
 			(at 55.5752 189.23 0)
 			(hide yes)

Commit message: replaced RECOM with AP63205WU-7 for better availability
Parts:
- removed U1: R-78E5.0-1.0, Converter_DCDC:Converter_DCDC_RECOM_R-78E-0.5_THT, symbol Converter_DCDC:R-78E5.0-1.0
- added C19: 22uF, Capacitor_SMD:C_1206_3216Metric, symbol Device:C
- added C20: 100nF, Capacitor_SMD:C_0805_2012Metric, symbol Device:C
- added L1: 4.7uH, Inductor_SMD:L_Sunlord_SWPA5040S, symbol Device:L
- added U1: AP63205WU-7, OpenFlipdisc_EasyEDA:TSOT-23-6_L2.9-W1.6-P0.95-LS2.8-BL, symbol OpenFlipdisc_EasyEDA:AP63205WU-7
Connections:
- net +5V: now also C19.1, L1.2, U1.1 (FB)
- net GND: now also C19.2, U1.4 (GND)
- net VM: now also U1.2 (EN), U1.3 (VIN)
- new net: C20.2, L1.1, U1.5 (SW)
- new net: C20.1, U1.6 (BST)
Other:
- moved on the sheet: A1, C1, C15, C16, C17, C18, C2, C3, C4, C5, D1, D2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
